Commit message: scales insoles now

File: urdf/insoles.urdf.xacro (robot description, xacro)
@@ -16,5 +16,5 @@
 		</joint>
 	</xacro:macro>
-	<xacro:macro name="insole_link" params="insole_name stl_name">
+	<xacro:macro name="insole_link" params="insole_name stl_name global_scale">
 		<link name="${insole_name}" >
 			<inertial>
@@ -38,5 +38,7 @@
 				<geometry>
 					<mesh
-						filename="package://moticon_insoles/meshes/${stl_name}" />
+						filename="package://moticon_insoles/meshes/${stl_name}"
+						scale = "${global_scale} ${global_scale} ${global_scale}"
+						/>
 				</geometry>
 				<material name="">
@@ -50,10 +52,12 @@
 				<geometry>
 					<mesh
-						filename="package://moticon_insoles/meshes/${stl_name}" />
+						filename="package://moticon_insoles/meshes/${stl_name}"
+						scale = "${global_scale} ${global_scale} ${global_scale}"
+						/>
 				</geometry>
 			</collision>
 		</link>
 	</xacro:macro>
-	<xacro:macro name="insole_joint" params="insole_name parent origin jtype">
+	<xacro:macro name="insole_joint" params="insole_name parent origin jtype global_scale">
 		<joint name="${insole_name}_joint" type="${jtype}">
 			<origin xyz="${origin}" rpy="0 0 0"/>
@@ -62,10 +66,13 @@
 		</joint>
 	</xacro:macro>
-	<xacro:macro name="insole_link_and_joint" params="parent origin side stl_name jtype">
-		<xacro:insole_link insole_name="${side}_insole" stl_name="${stl_name}"/>
+	<xacro:macro name="insole_link_and_joint" params="parent origin side stl_name jtype insole_scale_factor">
+		<xacro:insole_link insole_name="${side}_insole" stl_name="${stl_name}"
+			global_scale="${insole_scale_factor}"
+			/>
 		<xacro:insole_joint
 			insole_name="${side}_insole"
 			parent="${parent}"
 			origin="${origin}"
+			global_scale="${insole_scale_factor}"
 			jtype="${jtype}"/>
 	</xacro:macro>
